Commit message: Added velocity control, finger articulation, and touch sensors.

File: lyra_gz/models/hand_on_aion.xacro (robot description, xacro)
@@ -4,7 +4,6 @@
 	<!--Simple elevation arm-->
 	<link name="arm_link">
-		<origin xyz="0 0 0.15" rpy="0 0 0"/>
 		<collision name='arm_link_C'>
-			<origin xyz="0 0 0" rpy="0 0 0" />
+			<origin xyz="0 0 0.15" rpy="0 0 0" />
 			<geometry>
 				<box size=".03 .03 .3"/>
@@ -12,5 +11,5 @@
 		</collision>
 		<visual name='arm_link_V'>
-			<origin xyz="0 0 0" rpy="0 0 0" />
+			<origin xyz="0 0 0.15" rpy="0 0 0" />
 			<geometry>
 				<box size=".03 .03 .3"/>
@@ -18,4 +17,5 @@
 		</visual>
 		<inertial>
+			<origin xyz="0 0 0.15" rpy="0 0 0"/>
 			<mass value="0.014" />
 			<inertia
@@ -27,6 +27,6 @@
 	</link>
 	<joint name="arm_joint" type="revolute">
-		<origin xyz="0.2 0 0.2" rpy="1.57 1.57 1.57"/>
-		<axis xyz="1 0 0"/>
+		<origin xyz="0.15 0 0.15" rpy="1.57 1.57 1.57"/>
+		<axis xyz="0 1 0"/>
 		<limit lower="-1.5707" upper="1.5707" velocity="5.0" effort="1000"/>
 		<parent link="odom"/>
@@ -50,4 +50,4 @@
 	</gazebo>
 	<!--Hand-->
-	<xacro:include filename="$(find lyra_gz)/models/modularized_hand.urdf"/>
+	<xacro:include filename="$(find lyra_gz)/models/hand_module.urdf"/>
 </robot>

Commit message: Added arm hinge visual.

File: lyra_gz/models/hand_on_aion.xacro (robot description, xacro)
@@ -16,4 +16,10 @@
 			</geometry>
 		</visual>
+		<visual name="arm_link_pivot">
+			<origin xyz="0 0 0" rpy="0 1.57 1.57" />
+			<geometry>
+				<cylinder radius="0.03" length="0.1"/>
+			</geometry>
+		</visual>
 		<inertial>
 			<origin xyz="0 0 0.15" rpy="0 0 0"/>
@@ -27,5 +33,5 @@
 	</link>
 	<joint name="arm_joint" type="revolute">
-		<origin xyz="0.15 0 0.15" rpy="1.57 1.57 1.57"/>
+		<origin xyz="0.15 0 0.14" rpy="1.57 1.57 1.57"/>
 		<axis xyz="0 1 0"/>
 		<limit lower="-1.5707" upper="1.5707" velocity="5.0" effort="1000"/>
